File: BreadboardSchematic/MusicPlayer.kicad_sch (KiCad schematic)
At the start: 0 parts

Commit message: Added datasheets and finished the breadboard schematic
Parts:
- added C2, C3: 150nF, symbol Device:C
- added J1: VS1053b Module, symbol Connector_Generic_Shielded:Conn_02x14_Counter_Clockwise_Shielded
- added J2: SSD1306 Module, symbol Connector_Generic:Conn_01x04
- added R1, R2, R3, R4: 10k, symbol Device:R_US
- added SW1: RotaryEncoder, symbol Device:RotaryEncoder
- added SW2: Previous Track, symbol Switch:SW_Push
- added SW3: Next Track, symbol Switch:SW_Push
- added SW4: Play/Pause, symbol Switch:SW_Push
- added U1: STM32G031K8T6, Package_QFP:LQFP-32_7x7mm_P0.8mm, symbol MCU_ST_STM32G0:STM32G031K8Tx
Connections:
- new net: R2.1, R3.1, SW1.B
- new net: R1.2, R4.2, SW1.A
- new net +3V3: J1.gnd (Pin_4), J2.2 (3v3), R1.1, R2.2, SW2.2, SW3.1, SW4.2, U1.4 (VDD)
- new net Command Select: J1.XDCS (Pin_22), U1.15 (PB0)
- new net Data Request: J1.DREQ (Pin_21), U1.16 (PB1)
- new net Data Select: J1.MP3CS (Pin_20), U1.26 (PA15)
- new net Encoder A: C2.1, R4.1, U1.8 (PA1)
- new net Encoder B: C3.2, R3.2, U1.7 (PA0)
- new net GND: C2.2, C3.1, J1.3.3v (Pin_2), J2.1 (GND), SW1.C, U1.5 (VSS)
- new net I2C SCL: J2.3 (SCL), U1.30 (PB6)
- new net I2C SDA: J2.4 (SDA), U1.31 (PB7)
- new net Next Track: SW3.2, U1.29 (PB5)
- new net Play/Pause: SW4.1, U1.27 (PB3)
- new net Previous Track: SW2.1, U1.28 (PB4)
- new net SD Card Chip Select: J1.SDCS (Pin_19), U1.1 (PB9)
- new net SPI1 M0SI: U1.14 (PA7)
- new net SPI1 MISO: U1.13 (PA6)
- new net SPI1 SCK: J1.MISO (Pin_13), J1.MOSI (Pin_12), J1.SCLK (Pin_11), U1.12 (PA5)
- new net VCP RX: U1.9 (PA2)
- new net VCP TX: U1.10 (PA3)
- no-connect marks 0 -> 30
