File: PCB/Power.kicad_sch (KiCad schematic)
At the start: 32 parts, among them J1 3.7v LiPo, Q1 MMBT2907ALT1HTSA1, Q2 NMOS, U1 TPS61090, U2 LD1117S33TR_SOT223, U3 MCP73831T-2ACI/OT, U6 MAX17048G

Commit message: Finished making a PCB for it
Parts:
- R10: LCSC (none) -> C844915
Changed lines of the file:
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@@
+			)
+		)
+		(property "LCSC" "C844915"
+			(at 38.1 72.39 0)
+			(effects
+				(font
+					(size 1.27 1.27)
+				)
+				(hide yes)
 			)
 		)
